Commit message: Seems my changes to the urdf files weren't actually commited before. Previous fixes have been re-applied

File: scenes/hubo-models/huboplus.urdf (robot description, URDF)
Before this commit: robot huboplus, 58 links, 57 joints
Joints:
- joint RSR: limit lower=-1.5708 upper=1.5708 effort=10.0 velocity=1.0 -> lower=-1.5708 upper=0 effort=10.0 velocity=1.0
